File: PLC Kicad/PLC.kicad_pcb (KiCad board)
At the start: 2 copper layers, 128 parts, among them J1 24V, J10 TB_1X2, J11 Salida, J12 TB_1X2, J13 TB_1X2, J2 TB_1X2, J3 Salida, J4 Salida, J5 Salida, J6 Salida, J7 Salida, J8 Screw_Terminal_01x04, J9 TB_1X2, K1 RELAY_C, K2 RELAY_C, K3 RELAY_C, K4 RELAY_C, K5 RELAY_C, K7 RELAY_C, Q1 2N3904, Q10 2N3904, Q2 2N3904, Q3 2N3904, Q4 2N3904, Q5 2N3904, Q7 AO3401A, Q8 AO3401A, Q9 AO3401A, U1 LM2594M-5.0, U10 PC817, U11 BluePill, U12 SN74HC541PWR, U13 PC817, U14 PC817, U15 PC817, U16 PC817, U17 PC817, U2 LM2594M-3.3, U3 PC817, U4 PC817, U5 SN74HC14PWR, U6 PC817, U7 PC817, U8 PC817, U9 PC817

Commit message: Revisión 0.5 (PCB)
Parts:
- R10, R2, R4, R44, R6, R8: footprint Resistor_SMD:R_1210_3225Metric_Pad1.30x2.65mm_HandSolder -> EESTN5:RES0.3
- moved C10 443.4 mm to (-245.8, 216.6)
- moved C11 443.4 mm to (-245.8, 219.7)
- moved C12 443.4 mm to (-245.8, 222.7)
- moved C7 443.4 mm to (-228.9, 205.4)
- moved C8 443.4 mm to (-238.9, 205.9)
- moved C9 443.4 mm to (-245.8, 213.6)
- moved D16 443.4 mm to (-243.7, 226.5)
- moved D17 443.4 mm to (-243.7, 231.1)
- moved D18 443.4 mm to (-243.7, 235.8)
- moved J12 443.4 mm to (-269.2, 263.5)
- moved J13 443.4 mm to (-269.2, 274.7)
- moved J2 443.4 mm to (-205.4, 259.4)
- moved LED2 443.4 mm to (-260.5, 209.7)
- moved LED3 443.4 mm to (-260.5, 216.4)
- moved LED4 443.4 mm to (-260.5, 223.1)
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- renumbered K7 to K6
Connections:
- Q1 pad 1: GND -> Earth
- Q10 pad 1: GND -> Earth
- Q2 pad 1: GND -> Earth
- Q3 pad 1: GND -> Earth
- Q4 pad 1: GND -> Earth
- Q5 pad 1: GND -> Earth
- R10 pad 1: unconnected-(R10-Pad1) -> /PA01
- R2 pad 1: unconnected-(R2-Pad1) -> /PB07
- R4 pad 1: unconnected-(R4-Pad1) -> /PB08
- R44 pad 1: /PA0 -> /PA02
- R6 pad 1: unconnected-(R6-Pad1) -> /PB09
- R8 pad 1: unconnected-(R8-Pad1) -> /PA0
- U11 pad 15: unconnected-(U11-PB7-Pad15) -> /PB07
- U11 pad 16: unconnected-(U11-PB8-Pad16) -> /PB08
- U11 pad 17: unconnected-(U11-PB9-Pad17) -> /PB09
- U11 pad 26: unconnected-(U11-PA1-Pad26) -> /PA01
- U11 pad 27: unconnected-(U11-PA2-Pad27) -> /PA02
Routing:
- net 5V: track 248.1 -> 162.0 mm
- net /PA02: track 0.00 -> 71.4 mm
- net /PB07: track 0.00 -> 66.7 mm
- net /PB08: track 0.00 -> 52.0 mm
- net /PA01: track 0.00 -> 45.8 mm
- net Net-(J5-Pin_1): track 40.8 -> 0.00 mm
- net Net-(J11-Pin_1): track 40.7 -> 0.00 mm
- net Net-(J6-Pin_1): track 40.6 -> 0.00 mm
- net Net-(J4-Pin_1): track 40.6 -> 0.00 mm
- net Net-(J8-Pin_3): track 0.00 -> 40.6 mm
- net Net-(J7-Pin_1): track 40.6 -> 0.00 mm
- net Net-(J3-Pin_1): track 40.5 -> 0.00 mm
- net Net-(J8-Pin_4): track 0.00 -> 38.7 mm
- net /PB09: track 0.00 -> 26.0 mm
- net Net-(J8-Pin_2): track 0.00 -> 21.5 mm
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- added copper zone on F.Cu, net Earth
- added copper zone on F.Cu, net GND
