File: PLC Kicad/PLC.kicad_pcb (KiCad board)
At the start: 2 copper layers, 71 parts, among them J1 TB_1X2, J10 TB_1X2, J11 Salida, J2 TB_1X3, J3 Salida, J4 Salida, J5 Salida, J6 Salida, J7 Salida, J8 Screw_Terminal_01x04, J9 TB_1X2, K1 RELAY_C, K2 RELAY_C, K3 RELAY_C, K4 RELAY_C, K5 RELAY_C, K7 RELAY_C, Q1 2N3904, Q10 2N3904, Q2 2N3904, Q3 2N3904, Q4 2N3904, Q5 2N3904, Q7 AO3401A, Q8 AO3401A, Q9 AO3401A, U10 PC817, U4 PC817, U6 PC817, U7 PC817, U8 PC817, U9 PC817

Commit message: Revisión 0.3 (PCB)
primera fase de la PCB
Parts:
- added C10: C, Capacitor_SMD:C_0805_2012Metric_Pad1.18x1.45mm_HandSolder, F.Cu at (127.1, -23.2)
- added C11: C, Capacitor_SMD:C_0805_2012Metric_Pad1.18x1.45mm_HandSolder, F.Cu at (127.1, -20.2)
- added C12: C, Capacitor_SMD:C_0805_2012Metric_Pad1.18x1.45mm_HandSolder, F.Cu at (127.1, -17.2)
- added C7: C, Capacitor_SMD:C_0805_2012Metric_Pad1.18x1.45mm_HandSolder, F.Cu at (144.0, -34.5)
- added C8: C, Capacitor_SMD:C_0805_2012Metric_Pad1.18x1.45mm_HandSolder, F.Cu at (134.0, -34.0)
- added C9: C, Capacitor_SMD:C_0805_2012Metric_Pad1.18x1.45mm_HandSolder, F.Cu at (127.1, -26.2)
- added D1: 1N5822, Diode_THT:D_DO-201AD_P15.24mm_Horizontal, F.Cu at (-99.0, 151.1)
- added D16: 1N4148, M7:DIOM505270X240, F.Cu at (129.1, -13.4)
- added D17: 1N4148, M7:DIOM505270X240, F.Cu at (129.1, -8.74)
- added D18: 1N4148, M7:DIOM505270X240, F.Cu at (129.1, -4.09)
- added D2: 1N5822, Diode_THT:D_DO-201AD_P15.24mm_Horizontal, F.Cu at (-92.2, 151.1)
- added D3: SS210, SS210:DIOM4336X265N, F.Cu at (-83.8, 169.5)
- added D4: SS210, SS210:DIOM4336X265N, F.Cu at (-75.8, 169.5)
- added D5: SS210, SS210:DIOM4336X265N, F.Cu at (-75.8, 174.5)
- added D6: SS210, SS210:DIOM4336X265N, F.Cu at (-83.8, 174.5)
- added J12: TB_1X2, EESTN5:BORNERA2, F.Cu at (103.6, 23.6)
- added J13: TB_1X2, EESTN5:BORNERA2, F.Cu at (103.6, 34.8)
- added L1: 68uH, Inductor_SMD:L_Bourns_SRR1260, F.Cu at (-57.1, 165.5)
- added L2: 68uH, Inductor_SMD:L_Bourns_SRR1260, F.Cu at (-41.2, 165.5)
- added LED2: LED, EESTN5:led_5mm_green, F.Cu at (112.3, -30.2)
- added LED3: LED, EESTN5:led_5mm_green, F.Cu at (112.3, -23.5)
- added LED4: LED, EESTN5:led_5mm_green, F.Cu at (112.3, -16.8)
- added LED5: LED, EESTN5:led_5mm_green, F.Cu at (112.3, -10.1)
- added LED6: LED, EESTN5:led_5mm_green, F.Cu at (112.3, -3.43)
- added LED7: LED, EESTN5:led_5mm_green, F.Cu at (112.3, 3.27)
- added OK7: PC817, PC817X2NIP0F:SOP254P975X460-4N, F.Cu at (129.5, 10.7)
- added OK8: PC817, PC817X2NIP0F:SOP254P975X460-4N, F.Cu at (129.5, 19.2)
- added OK9: PC817, PC817X2NIP0F:SOP254P975X460-4N, F.Cu at (129.5, 27.8)
- added R12: R, EESTN5:R_0805, F.Cu at (76.0, -31.4)
- added R13: R, EESTN5:R_0805, F.Cu at (76.0, -26.6)
- added R14: R, EESTN5:R_0805, F.Cu at (76.0, -21.9)
- added R15: R, EESTN5:R_0805, F.Cu at (76.0, -17.1)
- added R16: R, EESTN5:R_0805, F.Cu at (76.0, -12.4)
- added R17: R, EESTN5:R_0805, F.Cu at (76.0, -7.65)
- added R18: R, EESTN5:R_0805, F.Cu at (76.0, -2.90)
- added R19: R, EESTN5:R_0805, F.Cu at (76.0, 1.85)
- added R20: R, EESTN5:R_0805, F.Cu at (76.0, 6.60)
- added R21: R, EESTN5:R_0805, F.Cu at (76.0, 11.3)
- added R22: R, EESTN5:R_0805, F.Cu at (76.0, 16.1)
- added R23: R, EESTN5:R_0805, F.Cu at (76.0, 20.9)
- added R24: R, EESTN5:R_0805, F.Cu at (76.0, 25.6)
- added R25: R, EESTN5:R_0805, F.Cu at (76.0, 30.4)
- added R26: R, EESTN5:R_0805, F.Cu at (76.0, 35.1)
- added R27: R, EESTN5:R_0805, F.Cu at (76.0, 39.9)
- added R28: R, EESTN5:R_0805, F.Cu at (76.0, 44.6)
- added R29: R, EESTN5:R_0805, F.Cu at (76.0, 49.4)
- added U1: LM2594M-5.0, LM2594M-5.0:SOIC127P599X175-8N, F.Cu at (-83.2, 161.5)
- added U12: SN74HC541PWR, SN74HC541PWR:SOP65P640X120-20N, F.Cu at (123.2, 45.1)
- added U13: PC817, Package_DIP:DIP-4_W7.62mm, F.Cu at (99.6, -25.0)
- added U14: PC817, Package_DIP:DIP-4_W7.62mm, F.Cu at (99.6, -18.3)
- added U15: PC817, Package_DIP:DIP-4_W7.62mm, F.Cu at (99.6, -11.6)
- added U16: PC817, Package_DIP:DIP-4_W7.62mm, F.Cu at (99.6, -4.90)
- added U17: PC817, Package_DIP:DIP-4_W7.62mm, F.Cu at (99.6, 1.80)
- added U2: LM2594M-3.3, LM2594M-3.3:SOIC127P599X175-8N, F.Cu at (-70.8, 161.5)
- added U3: PC817, Package_DIP:DIP-4_W7.62mm, F.Cu at (99.6, -31.7)
- added U5: SN74HC14PWR, SN74HC14PWR:SOP65P640X120-14N, F.Cu at (123.2, 37.8)
- C1, C4: value CP -> 470uF
- C2, C5: value C -> 1uF
- C3, C6: value CP -> 220uF
- J1: value TB_1X2 -> 24V
- J2: value TB_1X3 -> TB_1X2; footprint EESTN5:BORNERA3_AZUL -> EESTN5:BORNERA2
- LED1: footprint EESTN5:led_5mm_green -> LED_SMD:LED_0805_2012Metric
- R1: value R -> 1K
- R32, R33, R34, R35, R38, R39: footprint Resistor_THT:R_Axial_DIN0309_L9.0mm_D3.2mm_P20.32mm_Horizontal -> EESTN5:R_0805
- moved K1 252.8 mm to (24.4, 262.5), turned to 90 degrees
- moved K2 235.3 mm to (24.4, 245.5), turned to 90 degrees
- moved K3 219.0 mm to (24.4, 228.5), turned to 90 degrees
- moved K4 204.2 mm to (24.4, 211.5), turned to 90 degrees
- moved J1 193.5 mm to (-108.5, 159.1), turned to -90 degrees
- moved K5 191.3 mm to (24.4, 194.5), turned to 90 degrees
- moved K7 180.8 mm to (24.4, 177.5), turned to 90 degrees
- moved C3 171.9 mm to (-83.0, 149.2)
- moved C1 170.4 mm to (-72.8, 149.2)
- moved C2 168.9 mm to (-72.5, 154.2)
- moved LED1 162.8 mm to (-36.0, 147.5), turned to 90 degrees
- moved J2 159.9 mm to (167.5, 19.5)
- moved C5 153.8 mm to (-56.5, 154.2)
- moved C4 147.5 mm to (-56.7, 149.2)
- moved C6 134.4 mm to (-46.2, 149.2)
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Connections:
- C1 pad 1: Earth -> Net-(D2-K)
- C2 pad 1: Earth -> Net-(D2-K)
- C3 pad 1: /+5V -> Net-(U1-FB)
- J2 pad 1: unconnected-(J2-Pad1) -> /IN5
- J2 pad 2: unconnected-(J2-Pad2) -> /IN6
Routing:
- net Net-(U2-VIN): track 0.00 -> 79.4 mm
- net Net-(U2-OUT): track 0.00 -> 78.8 mm
- net Net-(U1-FB): track 0.00 -> 77.5 mm
- net /VCC: track 0.00 -> 69.1 mm
- net Net-(D2-K): track 0.00 -> 49.8 mm
- net Net-(U1-OUT): track 0.00 -> 31.9 mm
- net Net-(D2-A): track 0.00 -> 23.7 mm
- net Earth: track 0.00 -> 20.4 mm
- net 5V: track 0.00 -> 13.4 mm, vias 0 -> 1
- net Net-(LED1-A): track 0.00 -> 3.03 mm
- added copper zone on F.Cu, net Earth

Commit message: Revisión 0.4 (PCB)
Parts:
- added U11: BluePill, EESTN5:BluePill, F.Cu at (-106.1, 226.8)
- moved D10 226.9 mm to (-10.8, 267.9), turned to 90 degrees
- moved J3 210.9 mm to (28.0, 262.7), turned to 90 degrees
- moved U6 207.2 mm to (-30.9, 259.9), turned to -90 degrees
- moved D11 205.0 mm to (-10.8, 249.6), turned to 90 degrees
- moved R2 200.5 mm to (-39.2, 259.9)
- moved R3 194.7 mm to (-23.8, 263.8), turned to 180 degrees
- moved Q1 184.8 mm to (-17.0, 262.8)
- moved J4 184.5 mm to (28.0, 244.7), turned to 90 degrees
- moved D12 183.6 mm to (-10.8, 231.7), turned to 90 degrees
- moved U7 182.1 mm to (-30.9, 241.5), turned to -90 degrees
- moved R4 176.1 mm to (-39.2, 241.6)
- moved R6 170.0 mm to (-39.2, 223.1)
- moved R5 169.3 mm to (-23.8, 245.2), turned to 180 degrees
- moved R7 162.9 mm to (-23.8, 227.2), turned to 180 degrees
- moved D13 162.2 mm to (-10.8, 213.6), turned to 90 degrees
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Connections:
- R44 pad 1: unconnected-(R44-Pad1) -> /PA0
Routing:
- net 5V: track 13.4 -> 248.1 mm
- net /PA0: track 0.00 -> 50.8 mm
- net Net-(J5-Pin_1): track 0.00 -> 40.8 mm
- net Net-(J11-Pin_1): track 0.00 -> 40.7 mm
- net Net-(J6-Pin_1): track 0.00 -> 40.6 mm
- net Net-(J4-Pin_1): track 0.00 -> 40.6 mm
- net Net-(J7-Pin_1): track 0.00 -> 40.6 mm
- net Net-(J3-Pin_1): track 0.00 -> 40.5 mm
- net Net-(J5-Pin_3): track 0.00 -> 32.8 mm
- net Net-(J4-Pin_3): track 0.00 -> 32.8 mm
- net Net-(J3-Pin_3): track 0.00 -> 32.8 mm
- net Net-(J7-Pin_3): track 0.00 -> 32.6 mm
- net Net-(J6-Pin_3): track 0.00 -> 32.6 mm
- net Net-(J11-Pin_3): track 0.00 -> 32.5 mm
- net Net-(D13-K): track 0.00 -> 20.6 mm
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- removed copper zone on F.Cu, net Earth

Commit message: act pcb
hace que ocupe menos espacio
ahi te corregi unas cosas
Parts:
- removed D6: SS210, SS210:DIOM4336X265N
- added D7: SS210, Diode_SMD:D_SMA, F.Cu at (65.6, 26.1)
- added F1: Fuse, EESTN5:FUSIBLE, F.Cu at (91.6, 19.9)
- D1, D2: value 1N5822 -> SS210; footprint Diode_THT:D_DO-201AD_P15.24mm_Horizontal -> Diode_SMD:D_SMA
- D16, D17, D18: footprint M7:DIOM505270X240 -> EESTN5:DO-201AD
- D3, D4, D5: footprint SS210:DIOM4336X265N -> Diode_SMD:D_SMA
- OK7, OK8, OK9: footprint PC817X2NIP0F:SOP254P975X460-4N -> EESTN5:DIP-4_PC817
- U1: footprint LM2594M-5.0:SOIC127P599X175-8N -> EESTN5:SOIC-8_Hand_Soldering
- U17: footprint Package_DIP:DIP-4_W7.62mm -> EESTN5:DIP-4_PC817
- U2: footprint LM2594M-3.3:SOIC127P599X175-8N -> EESTN5:SOIC-8_Hand_Soldering
- moved J1 245.9 mm to (99.3, 27.7)
- moved JP1 234.3 mm to (-158.5, 36.6)
- moved Q8 234.3 mm to (-174.3, 35.0)
- moved Q9 234.3 mm to (-174.3, 39.6)
- moved J10 228.7 mm to (-229.8, 95.3)
- moved J8 228.7 mm to (-202.9, 100.6)
- moved J9 228.7 mm to (-229.8, 84.1)
- moved R32 228.7 mm to (-212.0, 69.3)
- moved R33 228.7 mm to (-212.2, 74.5)
- moved R34 228.7 mm to (-212.0, 78.8)
- moved R35 228.7 mm to (-212.0, 83.6)
- moved R36 228.7 mm to (-211.5, 109.0)
- moved R37 228.7 mm to (-211.5, 111.7)
- moved R38 228.7 mm to (-212.0, 88.3)
- moved R39 228.7 mm to (-212.0, 93.1)
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Connections:
- C1 pad 1: Net-(D2-K) -> Net-(D3-K)
- C2 pad 1: Net-(D2-K) -> Net-(D3-K)
- C3 pad 1: Net-(U1-FB) -> Net-(D2-A)
- C4 pad 1: Net-(U2-VIN) -> Net-(D4-K)
- C5 pad 1: Net-(U2-VIN) -> Net-(D4-K)
- D2 pad 1: Net-(D2-K) -> 5V
- L1 pad 1: Net-(U1-OUT) -> Net-(D7-K)
- L1 pad 2: Net-(U1-FB) -> Net-(D2-A)
- L2 pad 1: Net-(U2-OUT) -> Net-(D5-K)
- Q1 pad 1: GND -> Earth
- Q10 pad 1: GND -> Earth
- Q2 pad 1: GND -> Earth
- Q3 pad 1: GND -> Earth
- Q4 pad 1: GND -> Earth
- Q5 pad 1: GND -> Earth
- U1 pad 4: Net-(U1-FB) -> Net-(D2-A)
- U1 pad 7: Net-(D2-K) -> Net-(D3-K)
- U1 pad 8: Net-(U1-OUT) -> Net-(D7-K)
- U10 pad 2: GND -> Earth
- U11 pad 19: GND -> Earth
- U11 pad 39: GND -> Earth
- U11 pad 40: GND -> Earth
- U2 pad 7: Net-(U2-VIN) -> Net-(D4-K)
- U2 pad 8: Net-(U2-OUT) -> Net-(D5-K)
- U4 pad 2: GND -> Earth
- U6 pad 2: GND -> Earth
- U7 pad 2: GND -> Earth
- U8 pad 2: GND -> Earth
- U9 pad 2: GND -> Earth
Routing:
- net Earth: track 20.4 -> 603.4 mm, vias 0 -> 1
- net Net-(U2-VIN): track 79.4 -> 0.00 mm
- net Net-(U2-OUT): track 78.8 -> 0.00 mm
- net Net-(U1-FB): track 77.5 -> 0.00 mm
- net Net-(D7-K): track 0.00 -> 76.1 mm
- net Net-(D2-A): track 23.7 -> 89.3 mm
- net Net-(D2-K): track 49.8 -> 0.00 mm
- net /VCC: track 69.1 -> 27.2 mm
- net Net-(D3-K): track 0.00 -> 34.7 mm
- net Net-(U1-OUT): track 31.9 -> 0.00 mm
- net Net-(D5-K): track 0.00 -> 30.9 mm
- net /PA0: track 50.8 -> 77.2 mm
- net Net-(D4-K): track 0.00 -> 25.8 mm
- net Net-(F1-Pad1): track 0.00 -> 13.4 mm
- net Net-(R45-Pad2): track 20.0 -> 6.66 mm
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
Commit message: act1
..
Parts:
- added J14: Screw_Terminal_01x02, EESTN5:BORNERA2, F.Cu at (46.4, 113.3)
- C10, C11, C12, C9, R14, R15, R16, R17, R26, R27, R28, R29: moved to B.Cu
- J8: value Screw_Terminal_01x04 -> Screw_Terminal_01x02; footprint Library:Bornera_4 -> EESTN5:BORNERA2
- U12: value SN74HC541PWR -> PC817; footprint SN74HC541PWR:SOP65P640X120-20N -> Package_DIP:DIP-4_W7.62mm
- U16: value PC817 -> SN74HC14PWR; footprint Package_DIP:DIP-4_W7.62mm -> SN74HC14PWR:SOP65P640X120-14N
- U17: value PC817 -> SN74HC541PWR; footprint EESTN5:DIP-4_PC817 -> SN74HC541PWR:SOP65P640X120-20N
- U5: value SN74HC14PWR -> PC817; footprint SN74HC14PWR:SOP65P640X120-14N -> Package_DIP:DIP-4_W7.62mm
- moved J8 239.1 mm to (35.9, 113.4)
- moved JP1 225.2 mm to (53.3, 113.3), turned to 90 degrees
- moved U16 224.5 mm to (83.7, 146.2)
- moved R15 221.9 mm to (53.3, 140.4), turned to 180 degrees
- moved U17 218.4 mm to (84.5, 138.0)
- moved R17 212.2 mm to (53.0, 130.8), turned to 180 degrees
- moved R14 212.0 mm to (38.5, 140.3), turned to 180 degrees
- moved R16 201.3 mm to (38.3, 130.1), turned to 180 degrees
- moved R27 197.2 mm to (53.2, 138.0)
- moved U13 195.3 mm to (42.3, 135.7)
- moved R29 192.4 mm to (53.0, 128.4)
- moved R26 184.7 mm to (38.4, 138.1)
- moved R40 182.4 mm to (-47.7, 34.4)
- moved R41 182.4 mm to (-47.7, 37.1)
- moved R42 182.4 mm to (-47.7, 39.9)
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Connections:
- C10 pad 1: /4A hc14 -> /2A hc14
- C11 pad 1: /5A hc14 -> /3A hc14
- C12 pad 1: /6A hc14 -> /4A hc14
- C7 pad 1: /1A hc14 -> /5A hc14
- C8 pad 1: /2A hc14 -> /6A hc14
- C9 pad 1: /3A hc14 -> /1A hc14
- J13 pad 1: /IN1 -> /IN5
- J13 pad 2: /IN2 -> /IN6
- J2 pad 1: /IN5 -> /IN1
- J2 pad 2: /IN6 -> /IN2
- JP1 pad 1: Net-(J8-Pin_1) -> Net-(J14-Pin_1)
- JP1 pad 2: Net-(J8-Pin_2) -> Net-(J14-Pin_2)
- R12 pad 1: /IN1 -> /IN5
- R13 pad 1: /1A hc14 -> /IN6
- R13 pad 2: /VCC -> Net-(R13-Pad2)
- R14 pad 1: /1Y hc14 -> /IN1
- R14 pad 2: Net-(LED2-A) -> Net-(R14-Pad2)
- R16 pad 1: /2A hc14 -> /IN3
- R16 pad 2: /VCC -> Net-(R16-Pad2)
- R17 pad 1: /IN3 -> /IN4
- R18 pad 1: /3A hc14 -> /1Y hc14
- R18 pad 2: /VCC -> Net-(LED2-A)
- R19 pad 1: /IN4 -> /2Y hc14
- R19 pad 2: Net-(R19-Pad2) -> Net-(LED3-A)
- R20 pad 1: /4A hc14 -> /3Y hc14
- R20 pad 2: /VCC -> Net-(LED4-A)
- R21 pad 1: /IN5 -> /4Y hc14
- R21 pad 2: Net-(R21-Pad2) -> Net-(LED5-A)
- R22 pad 1: /5A hc14 -> /5Y hc14
- R22 pad 2: /VCC -> Net-(LED6-A)
- R23 pad 1: /IN6 -> /6Y hc14
- R23 pad 2: Net-(R23-Pad2) -> Net-(LED7-A)
- R24 pad 1: /6A hc14 -> /5A hc14
- R25 pad 1: /2Y hc14 -> /6A hc14
- R25 pad 2: Net-(LED3-A) -> /VCC
- R26 pad 1: /3Y hc14 -> /1A hc14
- R26 pad 2: Net-(LED4-A) -> /VCC
- R27 pad 1: /4Y hc14 -> /2A hc14
- R27 pad 2: Net-(LED5-A) -> /VCC
- R28 pad 1: /5Y hc14 -> /3A hc14
- R28 pad 2: Net-(LED6-A) -> /VCC
- R29 pad 1: /6Y hc14 -> /4A hc14
- R29 pad 2: Net-(LED7-A) -> /VCC
- U11 pad 15: unconnected-(U11-PB7-Pad15) -> /PB07
- U11 pad 16: unconnected-(U11-PB8-Pad16) -> /PB08
- U11 pad 17: unconnected-(U11-PB9-Pad17) -> /PB09
- U11 pad 19: Earth -> GND
- U11 pad 26: unconnected-(U11-PA1-Pad26) -> /PA01
- U11 pad 27: unconnected-(U11-PA2-Pad27) -> /PA02
- U11 pad 39: Earth -> GND
- U11 pad 40: Earth -> GND
- U11 pad 6: Net-(J8-Pin_4) -> Net-(J8-Pin_2)
- U11 pad 7: Net-(J8-Pin_3) -> Net-(J8-Pin_1)
- U12 pad 1: /1Y hc14 -> Net-(R14-Pad2)
- U12 pad 2: unconnected-(U12-1Y-Pad2) -> Earth
- U12 pad 3: /2Y hc14 -> Earth
- U12 pad 4: unconnected-(U12-2Y-Pad4) -> /1A hc14
- U14 pad 1: Net-(R17-Pad2) -> Net-(R16-Pad2)
- U15 pad 1: Net-(R19-Pad2) -> Net-(R17-Pad2)
- U16 pad 1: Net-(R21-Pad2) -> /1A hc14
- U16 pad 2: Earth -> /1Y hc14
- U16 pad 3: Earth -> /2A hc14
- U16 pad 4: /5A hc14 -> /2Y hc14
- U17 pad 1: Net-(R23-Pad2) -> /1Y hc14
- U17 pad 2: Earth -> unconnected-(U17-1Y-Pad2)
- U17 pad 3: Earth -> /2Y hc14
- U17 pad 4: /6A hc14 -> unconnected-(U17-2Y-Pad4)
- U3 pad 4: /1A hc14 -> /5A hc14
- U5 pad 1: /1A hc14 -> Net-(R13-Pad2)
- U5 pad 2: /1Y hc14 -> Earth
- U5 pad 3: /2A hc14 -> Earth
- U5 pad 4: /2Y hc14 -> /6A hc14
Routing:
- net 5V: track 240.1 -> 383.8 mm, vias 0 -> 1
- net /VCC: track 27.2 -> 111.8 mm, vias 0 -> 2
- net GND: track 0.00 -> 68.7 mm
- net Earth: track 603.4 -> 661.7 mm
- net /IN3: track 0.00 -> 44.6 mm
- net Net-(J8-Pin_2): track 0.00 -> 30.7 mm
- net /IN4: track 0.00 -> 27.7 mm
- net /IN2: track 0.00 -> 26.1 mm
- net Net-(J14-Pin_1): track 0.00 -> 24.9 mm
- net /IN1: track 0.00 -> 17.7 mm
- net Net-(J8-Pin_1): track 0.00 -> 16.5 mm
- net Net-(R16-Pad2): track 0.00 -> 13.5 mm
- net Net-(R17-Pad2): track 0.00 -> 13.5 mm
- net Net-(R15-Pad2): track 0.00 -> 13.3 mm
- net Net-(R14-Pad2): track 0.00 -> 13.1 mm
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