File: PLC Kicad/PLC.kicad_sch (KiCad schematic)
At the start: 129 parts, among them J1 24V, J10 TB_1X2, J11 Salida, J12 TB_1X2, J13 TB_1X2, J2 TB_1X2, J3 Salida, J4 Salida, J5 Salida, J6 Salida, J7 Salida, J8 Screw_Terminal_01x04, J9 TB_1X2, K1 RELAY_C, K2 RELAY_C, K3 RELAY_C, K4 RELAY_C, K5 RELAY_C, K7 RELAY_C, Q1 2N3904, Q10 2N3904, Q2 2N3904, Q3 2N3904, Q4 2N3904, Q5 2N3904, Q7 AO3401A, Q8 AO3401A, Q9 AO3401A, U1 LM2594M-5.0, U10 PC817, U11 BluePill, U12 SN74HC541PWR, U13 PC817, U14 PC817, U15 PC817, U16 PC817, U17 PC817, U2 LM2594M-3.3, U3 PC817, U4 PC817, U5 SN74HC14PWR, U6 PC817, U7 PC817, U8 PC817, U9 PC817

Commit message: Revisión 0.5 (PCB)
Parts:
- R10, R2, R4, R44, R6, R8: footprint Resistor_SMD:R_1210_3225Metric_Pad1.30x2.65mm_HandSolder -> EESTN5:RES0.3
- renumbered K7 to K6
Connections:
- net Earth: now also Q1.1 (E), Q10.1 (E), Q2.1 (E), Q3.1 (E), Q4.1 (E), Q5.1 (E); no longer U13.2, U14.2, U15.2, U16.2, U17.2, U3.2
- net GND: now also U13.2, U14.2, U15.2, U16.2, U17.2, U3.2; no longer Q1.1 (E), Q10.1 (E), Q2.1 (E), Q3.1 (E), Q4.1 (E), Q5.1 (E)
- net PA0: now also R8.1; no longer R44.1
- net PB08: now reaches R4.1
- net PB08: now also U11.16 (PB8)
- net PB07: now reaches R2.1
- net PB07: now also U11.15 (PB7)
- net PB09: now reaches R6.1
- net PB09: now also U11.17 (PB9)
- net PA01: now reaches U11.26 (PA1)
- net PA01: now also R10.1
- net PA02: now reaches U11.27 (PA2)
- net PA02: now also R44.1
Other:
- note removed: "GPIO"
- moved on the sheet: D10, D11, D12, D13, D14, D19, J11, J3, J4, J5, J6, J7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
