File: PLC Kicad/PLC.kicad_sch (KiCad schematic)
At the start: 25 parts, among them J1 TB_1X2, J2 TB_1X3, U1 LM2594M-5.0, U2 LM2594M-3.3, U3 LM321MF_NOPB, U5 LM321MF_NOPB

Commit message: revisión 0.1
Parts:
- added C7, C8, C9: C, symbol Device:C
- added D10, D11, D12, D13, D14, D15: 1N4148, Diode_THT:D_DO-35_SOD27_P7.62mm_Horizontal, symbol Diode:1N4148
- added D16, D17, D18: 1N4148, M7:DIOM505270X240, symbol Diode:1N4148
- added D8, D9: BZT52C3V3-7-F, BZT52C3V3-7-F:SOD3715X135N, symbol BZT52C3V3-7-F:BZT52C3V3-7-F
- added J10, J3, J4, J5, J6, J7, J8, J9: TB_1X2, EESTN5:BORNERA2, symbol EESTN5:TB_1X2
- added K1, K2, K3, K4, K5, K6: RELAY_C, SRD-24VDC-SL-C:RELAY_SRD-24VDC-SL-C, symbol EESTN5:RELAY_C
- added LED2, LED3, LED4, LED5, LED6, LED7: LED, symbol EESTN5:LED
- added OK1, OK2, OK3, OK4, OK5, OK6, OK7, OK8, OK9: PC817, PC817X2NIP0F:SOP254P975X460-4N, symbol PC817:PC817
- added Q1, Q2, Q3, Q4, Q5, Q6: MMBT3904, Package_TO_SOT_SMD:SOT-23, symbol Transistor_BJT:MMBT3904
- added Q7, Q8, Q9: AO3401A, Package_TO_SOT_SMD:SOT-23, symbol Transistor_FET:AO3401A
- added R10, R11, R12, R13, R14, R15, R16, R17, R18, R19, R20, R21, R22, R23, R24, R25, R26, R27, R28, R29, R3, R30, R31, R36, R37, R4, R40, R41, R42, R43, R5, R6, R7, R8, R9: R, EESTN5:R_0805, symbol Device:R
- added R32, R33, R34, R35, R38, R39: R, Resistor_THT:R_Axial_DIN0309_L9.0mm_D3.2mm_P20.32mm_Horizontal, symbol Device:R
- J1: footprint (none) -> EESTN5:BORNERA2
- J2: footprint (none) -> EESTN5:BORNERA3_AZUL
- LED1: footprint led 0805 -> (none)
- R1, R2: footprint (none) -> EESTN5:R_0805
Connections:
- net 24V: now also D10.1 (K), D11.1 (K), D12.1 (K), D13.1 (K), D14.1 (K), D15.1 (K), K1.5, K2.5, K3.5, K4.5, K5.5, K6.5, R11.1, R16.1, R21.1, R26.1, R31.1, R6.1
- net 5v1: now also OK1.4, OK2.4, OK3.4, OK4.4, OK5.4, OK6.4
- net Earth: now also C1.1, C2.1, D2.C, R2.1, U1.7 (VIN), D16.2 (A), D17.2 (A), D18.2 (A), J10.1, OK1.2, OK2.2, OK3.2, OK4.2, OK5.2, OK6.2, OK7.2, OK7.3, OK8.2, OK8.3, OK9.2, OK9.3, Q1.2 (E), Q2.2 (E), Q3.2 (E), Q4.2 (E), Q5.2 (E), Q6.2 (E), R12.1, R14.2, R17.1, R19.2, R22.1, R24.2, R27.1, R29.2, R32.1, R36.1, R40.1, R5.2, R7.1, R9.2
- net at R2.2: now also R3.1
- new net: Q6.1 (B), R30.2
- new net: D15.2 (A), K6.2, LED7.2 (K), Q6.3 (C)
- new net: J3.1, K1.1
- new net: D10.2 (A), K1.2, LED2.2 (K), Q1.3 (C)
- new net: J3.2, K1.3
- new net: OK2.3, R10.1, R9.1
- new net: R40.2, R41.1
- new net: R12.2, R13.1
- new net: OK3.1, R13.2
- new net: OK9.1, R41.2
- new net: Q4.1 (B), R20.2
- new net: D13.2 (A), K4.2, LED5.2 (K), Q4.3 (C)
- new net: Q2.1 (B), R10.2
- new net: OK8.4, R38.1, R39.1
- new net: Q8.3 (D), R38.2
- new net: OK6.3, R29.1, R30.1
- new net: R27.2, R28.1
- new net: OK1.3, R4.1, R5.1
- new net: Q1.1 (B), R4.2
- new net: R17.2, R18.1
- new net: OK4.1, R18.2
- new net: LED5.1 (A), R21.2
- new net: J6.1, K4.1
- new net: J6.2, K4.3
- new net: LED3.1 (A), R11.2
- new net: D11.2 (A), K2.2, LED3.2 (K), Q2.3 (C)
- new net: OK9.4, R42.1, R43.1
- new net: Q9.1 (G), R43.2
- new net: LED4.1 (A), R16.2
- new net: D12.2 (A), K3.2, LED4.2 (K), Q3.3 (C)
- new net: R22.2, R23.1
- new net: OK5.1, R23.2
- new net: J5.1, K3.1
- new net: J5.2, K3.3
- new net: J8.1, K6.1
- new net: J8.2, K6.3
- new net: J7.1, K5.1
- new net: D14.2 (A), K5.2, LED6.2 (K), Q5.3 (C)
- new net: J7.2, K5.3
- new net: OK3.3, R14.1, R15.1
- new net: OK8.1, R37.2
- new net: OK7.4, R34.1, R35.1
- new net: Q7.3 (D), R35.2
- new net: D18.1 (K), Q9.2 (S)
- new net: Q9.3 (D), R42.2
- new net: OK1.1, R3.2
- new net: Q8.1 (G), R39.2
- new net: OK4.3, R19.1, R20.1
- new net: R36.2, R37.1
- new net: OK6.1, R28.2
- new net: OK5.3, R24.1, R25.1
- new net: Q5.1 (B), R25.2
- new net: R32.2, R33.1
- new net: LED7.1 (A), R31.2
- new net: D16.1 (K), Q7.2 (S)
- new net: LED2.1 (A), R6.2
- new net: Q3.1 (B), R15.2
- new net: LED6.1 (A), R26.2
- new net: D17.1 (K), Q8.2 (S)
- new net: J4.1, K2.1
- new net: J4.2, K2.3
- new net: Q7.1 (G), R34.2
- new net: R7.2, R8.1
- new net: OK7.1, R33.2
- new net: OK2.1, R8.2
- no-connect marks 0 -> 6
Other:
- note added: "4/10/2025 (MM/DD/YYYY)"
- note added: "PLC"
- note added: "PWM outputs"
- note added: "Relay control"
- moved on the sheet: C1, C2, C3, C4, C5, C6, D1, D2, D3, D4, D5, D6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

Commit message: Librerias locales
modif Modulos rele
Librerias locales
-
Tenes que pasar las huellas y simbolos a librerias locales, asi el proyecto es portable
Parts:
- removed C7, C8, C9: C, symbol Device:C
- removed D10, D11, D12, D13, D14, D15: 1N4148, Diode_THT:D_DO-35_SOD27_P7.62mm_Horizontal, symbol Diode:1N4148
- removed D8, D9: BZT52C3V3-7-F, BZT52C3V3-7-F:SOD3715X135N, symbol BZT52C3V3-7-F:BZT52C3V3-7-F
- removed J2: TB_1X3, EESTN5:BORNERA3_AZUL, symbol EESTN5:TB_1X3
- removed J3, J4, J5, J6, J7, J8: TB_1X2, EESTN5:BORNERA2, symbol EESTN5:TB_1X2
- removed K6: RELAY_C, SRD-24VDC-SL-C:RELAY_SRD-24VDC-SL-C, symbol EESTN5:RELAY_C
- removed LED2, LED3, LED4, LED5, LED6, LED7: LED, symbol EESTN5:LED
- removed OK1, OK2, OK3, OK4, OK5, OK6: PC817, PC817X2NIP0F:SOP254P975X460-4N, symbol PC817:PC817
- removed Q1, Q2, Q3, Q4, Q5, Q6: MMBT3904, Package_TO_SOT_SMD:SOT-23, symbol Transistor_BJT:MMBT3904
- removed R12, R13, R14, R15, R16, R17, R18, R19, R20, R21, R22, R23, R24, R25, R26, R27, R28, R29, R30, R31: R, EESTN5:R_0805, symbol Device:R
- removed U3, U5: LM321MF_NOPB, LM321MF_NOPB:SOT95P280X145-5N, symbol LM321MF_NOPB:LM321MF_NOPB
- added D10, D11, D12, D13, D14, D19: 1N4007, Diode_THT:D_DO-41_SOD81_P10.16mm_Horizontal, symbol Diode:1N4007
- added J11, J3, J4, J5, J6, J7: Salida, EESTN5:BORNERA3_AZUL, symbol Connector:Screw_Terminal_01x03
- added J8: Screw_Terminal_01x04, Library:Bornera_4, symbol EESTN5:Screw_Terminal_01x04
- added JP1: Jumper, EESTN5:Jumper_Alto, symbol EESTN5:Jumper
- added K7: RELAY_C, EESTN5:Relay_C, symbol EESTN5:RELAY_C
- added Q1, Q10, Q2, Q3, Q4, Q5: 2N3904, Package_TO_SOT_SMD:SOT-23_Handsoldering, symbol Transistor_BJT:2N3904
- added R44: 220, Resistor_SMD:R_1210_3225Metric_Pad1.30x2.65mm_HandSolder, symbol Device:R
- added R45: 1k, Resistor_SMD:R_1210_3225Metric_Pad1.30x2.65mm_HandSolder, symbol Device:R
- added U10, U4, U6, U7, U8, U9: PC817, Package_DIP:DIP-4_W7.62mm, symbol EESTN5:PC817
- added U11: BluePill, EESTN5:BluePill_2, symbol EESTN5:BluePill
- C2, C5: footprint (none) -> Capacitor_SMD:C_0805_2012Metric_Pad1.18x1.45mm_HandSolder
- K1, K2, K3, K4, K5: footprint SRD-24VDC-SL-C:RELAY_SRD-24VDC-SL-C -> EESTN5:Relay_C
- LED1: footprint (none) -> EESTN5:led_5mm_green
- R10, R2, R4, R6, R8: value R -> 220; footprint EESTN5:R_0805 -> Resistor_SMD:R_1210_3225Metric_Pad1.30x2.65mm_HandSolder
- R11, R3, R5, R7, R9: value R -> 1k; footprint EESTN5:R_0805 -> Resistor_SMD:R_1210_3225Metric_Pad1.30x2.65mm_HandSolder
Connections:
- net 24V: no longer K1.5, K2.5, K3.5, K4.5, K5.5, R11.1, R6.1
- net Earth: no longer R2.1, R5.2, R7.1, R9.2
- net at K1.1: now also J3.3 (Pin_3)
- net at K1.2: now also D10.1 (K), Q1.3 (C)
- net at K1.3: now also J3.2 (Pin_2)
- net at K1.4: now also J3.1 (Pin_1)
- net at R9.1: now also Q4.2 (B); no longer R10.1
- net at K4.2: now also D13.1 (K), Q4.3 (C)
- net at R10.2: now also U10.1
- net at R5.1: now also Q2.2 (B); no longer R4.1
- net at R4.2: now also U7.1
- net at K4.1: now also J6.3 (Pin_3)
- net at K4.3: now also J6.2 (Pin_2)
- net at R11.2: now also U10.3
- net at K2.2: now also D11.1 (K), Q2.3 (C)
- net at K3.2: now also D12.1 (K), Q3.3 (C)
- net at R3.1: now also Q1.2 (B); no longer R2.2
- net at K3.1: now also J5.3 (Pin_3)
- net at K3.3: now also J5.2 (Pin_2)
- net at K5.1: now also J7.3 (Pin_3)
- net at K5.2: now also D14.1 (K), Q5.3 (C)
- net at K5.3: now also J7.2 (Pin_2)
- net at K5.4: now also J7.1 (Pin_1)
- net at R3.2: now also U6.3
- net at R6.2: now also U8.1
- net at K3.4: now also J5.1 (Pin_1)
- net at K2.1: now also J4.3 (Pin_3)
- net at K2.3: now also J4.2 (Pin_2)
- net at R7.2: now also U8.3; no longer R8.1
- net at K2.4: now also J4.1 (Pin_1)
- net at R8.2: now also U9.1
- net at K4.4: now also J6.1 (Pin_1)
- new net: R44.2, U4.1
- new net: R45.2, U4.3
- new net: Q10.2 (B), R45.1
- new net: D19.1 (K), K7.2, Q10.3 (C)
- new net: R5.2, U7.3
- new net: R2.2, U6.1
- new net: J8.1 (Pin_1), JP1.1 (A)
- new net: J8.2 (Pin_2), JP1.2 (B)
- new net: J8.3 (Pin_3), U11.7 (PA10)
- new net: J8.4 (Pin_4), U11.6 (PA9)
- new net: Q3.2 (B), R7.1
- new net: J11.1 (Pin_1), K7.4
- new net: J11.2 (Pin_2), K7.3
- new net: J11.3 (Pin_3), K7.1
- new net: Q5.2 (B), R11.1
- new net: R9.2, U9.3
- new net 5V: D10.2 (A), D11.2 (A), D12.2 (A), D13.2 (A), D14.2 (A), D19.2 (A), K1.5, K2.5, K3.5, K4.5, K5.5, K7.5, U10.4, U11.18 (5V), U4.4, U6.4, U7.4, U8.4, U9.4
- new net GND: Q1.1 (E), Q10.1 (E), Q2.1 (E), Q3.1 (E), Q4.1 (E), Q5.1 (E), U10.2, U11.19 (GND), U11.39 (GND), U11.40 (GND), U4.2, U6.2, U7.2, U8.2, U9.2
- no-connect marks 6 -> 0
Other:
- note added: "COM"
- note added: "DE"
- note added: "GPIO"
- note added: "NA"
- note added: "NC"
- note added: "RE"
- note added: "RX"
- note added: "Rele"
- note added: "STM32"
- note added: "TX"

Commit message: PLC (revisón 0.2)
Parts:
- added C10, C11, C12, C7, C8, C9: C, Capacitor_SMD:C_0805_2012Metric_Pad1.18x1.45mm_HandSolder, symbol Device:C
- added J12, J13, J2: TB_1X2, EESTN5:BORNERA2, symbol EESTN5:TB_1X2
- added LED2, LED3, LED4, LED5, LED6, LED7: LED, EESTN5:led_5mm_green, symbol EESTN5:LED
- added R12, R13, R14, R15, R16, R17, R18, R19, R20, R21, R22, R23, R24, R25, R26, R27, R28, R29: R, Resistor_THT:R_Axial_DIN0309_L9.0mm_D3.2mm_P20.32mm_Horizontal, symbol Device:R
- added U12: SN74HC541PWR, SN74HC541PWR:SOP65P640X120-20N, symbol SN74HC14PWR:SN74HC14PWR
- added U13, U14, U15, U16, U17, U3: PC817, Package_DIP:DIP-4_W7.62mm, symbol EESTN5:PC817
- added U5: SN74HC14PWR, SN74HC14PWR:SOP65P640X120-14N, symbol SN74HC14PWR:SN74HC14PWR
Connections:
- net Earth: now also LED2.2 (K), LED3.2 (K), LED4.2 (K), LED5.2 (K), LED6.2 (K), LED7.2 (K), U12.7 (GND), U13.2, U13.3, U14.2, U14.3, U15.2, U15.3, U16.2, U16.3, U17.2, U17.3, U3.2, U3.3, U5.7 (GND)
- net VCC: now also C10.2, C11.2, C12.2, C7.2, C8.2, C9.2, R13.2, R16.2, R18.2, R20.2, R22.2, R24.2, U12.14 (VCC), U5.14 (VCC)
- new net: LED3.1 (A), R25.2
- new net: R19.2, U15.1
- new net: R23.2, U17.1
- new net: R12.2, U3.1
- new net: LED2.1 (A), R14.2
- new net: LED6.1 (A), R28.2
- new net: R17.2, U14.1
- new net: LED5.1 (A), R27.2
- new net: R21.2, U16.1
- new net: R15.2, U13.1
- new net: LED4.1 (A), R26.2
- new net: LED7.1 (A), R29.2
- new net 1A hc14: C7.1, R13.1, U3.4, U5.1 (1A)
- new net 1Y hc14: R14.1, U12.1 (1A), U5.2 (1Y)
- new net 2A hc14: C8.1, R16.1, U13.4, U5.3 (2A)
- new net 2Y hc14: R25.1, U12.3 (2A), U5.4 (2Y)
- new net 3A hc14: C9.1, R18.1, U14.4, U5.5 (3A)
- new net 3Y hc14: R26.1, U12.5 (3A), U5.6 (3Y)
- new net 4A hc14: C10.1, R20.1, U15.4, U5.9 (4A)
- new net 4Y hc14: R27.1, U12.9 (4A), U5.8 (4Y)
- new net 5A hc14: C11.1, R22.1, U16.4, U5.11 (5A)
- new net 5Y hc14: R28.1, U12.11 (5A), U5.10 (5Y)
- new net 6A hc14: C12.1, R24.1, U17.4, U5.13 (6A)
- new net 6Y hc14: R29.1, U12.13 (6A), U5.12 (6Y)
- new net IN1: J13.1, R12.1
- new net IN2: J13.2, R15.1
- new net IN3: J12.1, R17.1
- new net IN4: J12.2, R19.1
- new net IN5: J2.1, R21.1
- new net IN6: J2.2, R23.1
Other:
- note added: "04/10/2025 (MM/DD/YYYY)"
- note added: "04/18/2025 (MM/DD/YYYY)"
- note added: "Digital inputs"
- note removed: "4/10/2025 (MM/DD/YYYY)"
- moved on the sheet: C1, C2, C3, C4, C5, C6, D1, D10, D11, D12, D13, D14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

Commit message: Revisión 0.3 (PCB)
primera fase de la PCB
Parts:
- removed D1, D2, D7: SS210, SS210:DIOM4336X265N, symbol SS210:SS210
- added D1, D2: 1N5822, Diode_THT:D_DO-201AD_P15.24mm_Horizontal, symbol Diode:1N5822
- C1, C4: value CP -> 470uF
- C2, C5: value C -> 1uF
- C3, C6: value CP -> 220uF
- J1: value TB_1X2 -> 24V
- L1, L2: value L -> 68uH; footprint (none) -> Inductor_SMD:L_Bourns_SRR1260
- LED1: footprint EESTN5:led_5mm_green -> LED_SMD:LED_0805_2012Metric
- R1: value R -> 1K
- R12, R13, R14, R15, R16, R17, R18, R19, R20, R21, R22, R23, R24, R25, R26, R27, R28, R29, R32, R33, R34, R35, R38, R39: footprint Resistor_THT:R_Axial_DIN0309_L9.0mm_D3.2mm_P20.32mm_Horizontal -> EESTN5:R_0805
Connections:
- net 24V is gone; now on an unnamed net: D3.C
- net 5v1 is gone; now on an unnamed net: D6.C
- net 5V: now also D5.C
- net Earth: now also D3.A, D6.A, D1.1 (K), D1.2 (A); no longer C1.1, C2.1, D4.A, U1.7 (VIN)
- net at F1.2: now also D2.2 (A); no longer D3.A
- net at L1.1, U1.8 (OUT): no longer D4.C
- net at C4.1, C5.1, U2.7 (VIN): now also D4.C; no longer D5.C
- net +5V: no longer names the net of C3.1, D5.A, L1.2, U1.4 (FB)
- net +5V: now also D4.A; no longer D6.A
- new net: C1.1, C2.1, D2.1 (K), U1.7 (VIN)

Commit message: Revisión 0.4 (PCB)
Parts:
- U11: footprint EESTN5:BluePill_2 -> EESTN5:BluePill
Connections:
- net PA0: now reaches R44.1
- net PA0: now also U11.25 (PA0)
Other:
- moved on the sheet: D10, D11, D12, D13, D14, D19, J11, J3, J4, J5, J6, J7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

Commit message: act pcb
hace que ocupe menos espacio
ahi te corregi unas cosas
Parts:
- removed D1, D2: 1N5822, Diode_THT:D_DO-201AD_P15.24mm_Horizontal, symbol Diode:1N5822
- removed D3, D4, D5, D6: SS210, SS210:DIOM4336X265N, symbol SS210:SS210
- added D1, D2, D3, D4, D5, D7: SS210, Diode_SMD:D_SMA, symbol Diode:SS210
- D16, D17, D18: footprint M7:DIOM505270X240 -> EESTN5:DO-201AD
- F1: footprint (none) -> EESTN5:FUSIBLE
- OK7, OK8, OK9: footprint PC817X2NIP0F:SOP254P975X460-4N -> EESTN5:DIP-4_PC817
- U1: footprint LM2594M-5.0:SOIC127P599X175-8N -> EESTN5:SOIC-8_Hand_Soldering
- U17: footprint Package_DIP:DIP-4_W7.62mm -> EESTN5:DIP-4_PC817
- U2: footprint LM2594M-3.3:SOIC127P599X175-8N -> EESTN5:SOIC-8_Hand_Soldering
Connections:
- net GND is gone; now on net Earth: Q1.1 (E), Q10.1 (E), Q2.1 (E), Q3.1 (E), Q4.1 (E), Q5.1 (E), U10.2, U11.19 (GND), U11.39 (GND), U11.40 (GND), U4.2, U6.2, U7.2, U8.2, U9.2
- net 5V: now also D2.1 (K)
- net Earth: now also D1.1 (K), D1.2 (A), D5.2 (A), D7.2 (A)
- net at F1.2: now also D3.2 (A)
- net at L2.1, U2.8 (OUT): now also D5.1 (K)
- net at C3.1, L1.2, U1.4 (FB): now also D2.2 (A), D4.2 (A)
- net at L1.1, U1.8 (OUT): now also D7.1 (K)
- net at C4.1, C5.1, U2.7 (VIN): now also D4.1 (K)
- net at C1.1, C2.1, U1.7 (VIN): now also D3.1 (K)

Commit message: act1
..
Parts:
- removed J8: Screw_Terminal_01x04, Library:Bornera_4, symbol EESTN5:Screw_Terminal_01x04
- removed U12: SN74HC541PWR, SN74HC541PWR:SOP65P640X120-20N, symbol SN74HC14PWR:SN74HC14PWR
- removed U16: PC817, Package_DIP:DIP-4_W7.62mm, symbol EESTN5:PC817
- removed U17: PC817, EESTN5:DIP-4_PC817, symbol EESTN5:PC817
- removed U5: SN74HC14PWR, SN74HC14PWR:SOP65P640X120-14N, symbol SN74HC14PWR:SN74HC14PWR
- added J14, J8: Screw_Terminal_01x02, EESTN5:BORNERA2, symbol Connector:Screw_Terminal_01x02
- added U12, U5: PC817, Package_DIP:DIP-4_W7.62mm, symbol EESTN5:PC817
- added U16: SN74HC14PWR, SN74HC14PWR:SOP65P640X120-14N, symbol SN74HC14PWR:SN74HC14PWR
- added U17: SN74HC541PWR, SN74HC541PWR:SOP65P640X120-20N, symbol SN74HC14PWR:SN74HC14PWR
Connections:
- net 1A hc14: now also C9.1, R26.1, U12.4, U16.1 (1A); no longer C7.1, R13.1, U3.4
- net 1Y hc14: now also R18.1, U16.2 (1Y), U17.1 (1A); no longer R14.1
- net 2A hc14: now also C10.1, R27.1, U16.3 (2A); no longer C8.1, R16.1
- net 2Y hc14: now also R19.1, U16.4 (2Y), U17.3 (2A); no longer R25.1
- net 3A hc14: now also C11.1, R28.1, U16.5 (3A); no longer C9.1, R18.1
- net 3Y hc14: now also R20.1, U16.6 (3Y), U17.5 (3A); no longer R26.1
- net 4A hc14: now also C12.1, R29.1, U16.9 (4A); no longer C10.1, R20.1
- net 4Y hc14: now also R21.1, U16.8 (4Y), U17.9 (4A); no longer R27.1
- net 5A hc14: now also C7.1, R24.1, U3.4, U16.11 (5A); no longer C11.1, R22.1
- net 5Y hc14: now also R22.1, U16.10 (5Y), U17.11 (5A); no longer R28.1
- net 6A hc14: now also C8.1, R25.1, U16.13 (6A), U5.4; no longer C12.1, R24.1
- net 6Y hc14: now also R23.1, U16.12 (6Y), U17.13 (6A); no longer R29.1
- net Earth: now also U12.2, U12.3, U16.7 (GND), U17.7 (GND), U5.2, U5.3; no longer U11.19 (GND), U11.39 (GND), U11.40 (GND)
- net IN1: now also J2.1, R14.1; no longer J13.1, R12.1
- net IN2: now also J2.2; no longer J13.2
- net IN3: now also R16.1; no longer R17.1
- net IN4: now also R17.1; no longer R19.1
- net IN5: now also J13.1, R12.1; no longer J2.1, R21.1
- net IN6: now also J13.2, R13.1; no longer J2.2, R23.1
- net VCC: now also R25.2, R26.2, R27.2, R28.2, R29.2, U16.14 (VCC), U17.14 (VCC); no longer R13.2, R16.2, R18.2, R20.2, R22.2
- net at LED3.1 (A): now also R19.2; no longer R25.2
- net at U15.1: now also R17.2; no longer R19.2
- net at R23.2: now also LED7.1 (A)
- net at R14.2: now also U12.1; no longer LED2.1 (A)
- net at LED6.1 (A): now also R22.2; no longer R28.2
- net at JP1.1 (A): now also J14.1 (Pin_1)
- net at JP1.2 (B): now also J14.2 (Pin_2)
- net at U11.7 (PA10): now also J8.1 (Pin_1)
- net at U11.6 (PA9): now also J8.2 (Pin_2)
- net at U14.1: now also R16.2; no longer R17.2
- net at LED5.1 (A): now also R21.2; no longer R27.2
- net PB07: now reaches U11.15 (PB7)
- net PB08: now reaches U11.16 (PB8)
- net PB09: now reaches U11.17 (PB9)
- net PA01: now reaches U11.26 (PA1)
- net PA02: now reaches U11.27 (PA2)
- net at LED4.1 (A): now also R20.2; no longer R26.2
- new net: LED2.1 (A), R18.2
- new net: R13.2, U5.1
- new net GND: U11.19 (GND), U11.39 (GND), U11.40 (GND)
