File: PLC Kicad 2/PLC-2025-05-02_231709/PLC.kicad_sch (KiCad schematic)
At the start: 129 parts, among them J1 24V, J10 TB_1X2, J11 Salida, J12 TB_1X2, J13 TB_1X2, J2 TB_1X2, J3 Salida, J4 Salida, J5 Salida, J6 Salida, J7 Salida, J8 Screw_Terminal_01x04, J9 TB_1X2, K1 RELAY_C, K2 RELAY_C, K3 RELAY_C, K4 RELAY_C, K5 RELAY_C, K6 RELAY_C, Q1 2N3904, Q10 2N3904, Q2 2N3904, Q3 2N3904, Q4 2N3904, Q5 2N3904, Q7 AO3401A, Q8 AO3401A, Q9 AO3401A, U1 LM2594M-5.0, U10 PC817, U11 BluePill, U12 SN74HC541PWR, U13 PC817, U14 PC817, U15 PC817, U16 PC817, U17 PC817, U2 LM2594M-3.3, U3 PC817, U4 PC817, U5 SN74HC14PWR, U6 PC817, U7 PC817, U8 PC817, U9 PC817

Commit message: Revision 0.6 (fin proto PCB)
Parts:
- C7, C8: value C -> 100nF; footprint Capacitor_SMD:C_0805_2012Metric_Pad1.18x1.45mm_HandSolder -> Capacitor_THT:C_Rect_L7.2mm_W2.5mm_P5.00mm_FKS2_FKP2_MKS2_MKP2
- R12, R15: value R -> 10K
- R13, R16: value R -> 10K; footprint EESTN5:R_0805 -> EESTN5:RES0.3
Connections:
- net PA01: now also U12.2 (1Y)
- net PA02: now also U12.4 (2Y); no longer R44.1
- net PB09: now also R44.1
- no-connect marks 0 -> 30

Commit message: Revision 0.7 (BUCKS)
Parts:
- added J14, J15, J16, J17: TB_1X2, EESTN5:BORNERA2, symbol EESTN5:TB_1X2
Connections:
- net 5V: now also J15.1, J16.1
- net Earth: now also J14.2, J15.2, J16.2, J17.2
- net VCC: now also J17.1
- new net + buck 5V: J14.1
Other:
- note added: "BUCKS 5V-3.3V"
